File: cagelock/cagelock.kicad_pcb (KiCad board)
At the start: 2 copper layers, 78.1 x 64.1 mm, 18 parts, among them J1 Conn_01x02, J2 Conn_01x04, J3 Conn_01x02, J4 Conn_01x02, J5 Conn_01x02, J6 Conn_01x02, J7 Conn_01x02, Q1 2N3904, U1 NodeMCU_v2

Commit message: correct pcb
Parts:
- moved J7 1.80 mm to (127.0, 141.0), turned to 0 degrees
Routing:
- net +3V3: track 30.3 -> 108.6 mm, vias 0 -> 1
- net GND: track 8.69 -> 65.5 mm
- net +12V: track 4.08 -> 46.8 mm
- net /DOOR_SENSE: track 0.00 -> 33.3 mm, vias 0 -> 1
Changed lines of the file:
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@@
     (thickness 1.6)
     (drawings 4)
-    (tracks 38)
+    (tracks 83)
     (zones 0)
     (modules 18)
@@
   )
   (setup
-    (last_trace_width 0.25)
+    (last_trace_width 1)
     (user_trace_width 1)
     (trace_clearance 0.2)
@@
   )
   (module Connector_PinHeader_2.54mm:PinHeader_1x02_P2.54mm_Vertical (layer F.Cu)
-    (at 128.27 142.24 180)
+    (at 127 140.97)
     (descr "Through hole straight pin header, 1x02, 2.54mm pitch, single row")
     (tags "Through hole pin header THT 1x02 2.54mm single row")
@@
       (effects (font (size 1 1) (thickness 0.15)))
     )
-    (pad 1 thru_hole rect (at 0 0 180) (size 1.7 1.7) (drill 1) (layers *.Cu *.Mask)
-      (net 2 GND))
-    (pad 2 thru_hole oval (at 0 2.54 180) (size 1.7 1.7) (drill 1) (layers *.Cu *.Mask)
+    (pad 1 thru_hole rect (at 0 0) (size 1.7 1.7) (drill 1) (layers *.Cu *.Mask)
+      (net 2 GND))
+    (pad 2 thru_hole oval (at 0 2.54) (size 1.7 1.7) (drill 1) (layers *.Cu *.Mask)
       (net 32 +5V))
     (model ${KISYS3DMOD}/Connector_PinHeader_2.54mm.3dshapes/PinHeader_1x02_P2.54mm_Vertical.wrl
@@
   (segment (start 152.4 114.3) (end 149.86 111.76) (width 1) (layer F.Cu) (net 2))
   (segment (start 154.31 114.3) (end 152.4 114.3) (width 1) (layer F.Cu) (net 2))
+  (segment (start 127 140.97) (end 139.7 140.97) (width 1) (layer F.Cu) (net 2))
+  (segment (start 140.97 142.24) (end 140.97 151.13) (width 1) (layer F.Cu) (net 2))
+  (segment (start 139.7 140.97) (end 140.97 142.24) (width 1) (layer F.Cu) (net 2))
+  (segment (start 156.21 151.13) (end 156.21 149.86) (width 1) (layer B.Cu) (net 2))
+  (segment (start 158.75 147.32) (end 160.02 147.32) (width 1) (layer B.Cu) (net 2))
+  (segment (start 161.29 148.59) (end 161.29 151.13) (width 1) (layer B.Cu) (net 2))
+  (segment (start 160.02 147.32) (end 161.29 148.59) (width 1) (layer B.Cu) (net 2))
+  (segment (start 157.48 148.59) (end 158.75 147.32) (width 1) (layer B.Cu) (net 2))
+  (segment (start 156.21 149.86) (end 157.48 148.59) (width 1) (layer B.Cu) (net 2))
+  (segment (start 140.97 147.32) (end 140.97 151.13) (width 1) (layer B.Cu) (net 2))
+  (segment (start 157.48 148.59) (end 153.67 144.78) (width 1) (layer B.Cu) (net 2))
+  (segment (start 143.51 144.78) (end 140.97 147.32) (width 1) (layer B.Cu) (net 2))
+  (segment (start 153.67 144.78) (end 143.51 144.78) (width 1) (layer B.Cu) (net 2))
   (segment (start 157.48 104.63) (end 160.02 107.17) (width 1) (layer F.Cu) (net 3))
   (segment (start 157.48 104.14) (end 157.48 104.63) (width 1) (layer F.Cu) (net 3))
+  (segment (start 154.94 104.14) (end 157.48 104.14) (width 1) (layer F.Cu) (net 3))
+  (segment (start 132.08 128.27) (end 147.32 113.03) (width 1) (layer F.Cu) (net 3))
+  (segment (start 147.32 113.03) (end 147.32 109.22) (width 1) (layer F.Cu) (net 3))
+  (segment (start 127 128.27) (end 132.08 128.27) (width 1) (layer F.Cu) (net 3))
+  (segment (start 147.32 109.22) (end 149.86 106.68) (width 1) (layer F.Cu) (net 3))
+  (segment (start 152.4 106.68) (end 154.94 104.14) (width 1) (layer F.Cu) (net 3))
+  (segment (start 149.86 106.68) (end 152.4 106.68) (width 1) (layer F.Cu) (net 3))
   (segment (start 157.48 111.76) (end 157.48 114.57) (width 1) (layer F.Cu) (net 4))
   (segment (start 160.02 109.22) (end 157.48 111.76) (width 1) (layer F.Cu) (net 4))
@@
   (segment (start 167.64 127) (end 166.37 125.73) (width 0.25) (layer F.Cu) (net 10))
   (segment (start 166.37 125.73) (end 163.83 125.73) (width 0.25) (layer F.Cu) (net 10))
-  (segment (start 184.34237 127) (end 167.64 127) (width 0.25) (layer F.Cu) (net 10))
   (segment (start 185.61237 128.27) (end 184.34237 127) (width 0.25) (layer F.Cu) (net 10))
   (segment (start 186.69 128.27) (end 185.61237 128.27) (width 0.25) (layer F.Cu) (net 10))
   (segment (start 186.69 128.27) (end 189.23 128.27) (width 0.25) (layer F.Cu) (net 10))
+  (segment (start 163.83 125.73) (end 159.38359 125.73) (width 0.25) (layer B.Cu) (net 10))
+  (segment (start 159.38359 125.73) (end 157.48 125.73) (width 0.25) (layer B.Cu) (net 10))
+  (segment (start 157.48 125.73) (end 151.13 132.08) (width 0.25) (layer B.Cu) (net 10))
+  (via (at 151.13 142.24) (size 0.8) (drill 0.4) (layers F.Cu B.Cu) (net 10))
+  (segment (start 151.13 132.08) (end 151.13 142.24) (width 0.25) (layer B.Cu) (net 10))
+  (segment (start 151.13 142.24) (end 151.13 140.97) (width 0.25) (layer F.Cu) (net 10))
+  (segment (start 151.13 140.97) (end 153.67 138.43) (width 0.25) (layer F.Cu) (net 10))
+  (segment (start 153.67 138.43) (end 154.94 138.43) (width 0.25) (layer F.Cu) (net 10))
+  (segment (start 154.94 138.43) (end 157.48 140.97) (width 0.25) (layer F.Cu) (net 10))
+  (segment (start 157.48 140.97) (end 157.48 143.51) (width 0.25) (layer F.Cu) (net 10))
+  (segment (start 155.72 145.27) (end 153.67 145.27) (width 0.25) (layer F.Cu) (net 10))
+  (segment (start 157.48 143.51) (end 155.72 145.27) (width 0.25) (layer F.Cu) (net 10))
+  (segment (start 176.53 104.14) (end 176.53 127) (width 0.25) (layer F.Cu) (net 10))
+  (segment (start 175.26 102.87) (end 176.53 104.14) (width 0.25) (layer F.Cu) (net 10))
+  (segment (start 163.83 102.87) (end 175.26 102.87) (width 0.25) (layer F.Cu) (net 10))
+  (segment (start 184.34237 127) (end 176.53 127) (width 0.25) (layer F.Cu) (net 10))
+  (segment (start 176.53 127) (end 167.64 127) (width 0.25) (layer F.Cu) (net 10))
   (segment (start 158.75 120.65) (end 158.75 128.27) (width 0.25) (layer F.Cu) (net 11))
   (segment (start 158.75 128.27) (end 161.29 130.81) (width 0.25) (layer F.Cu) (net 11))
   (segment (start 161.29 130.81) (end 162.56 130.81) (width 0.25) (layer F.Cu) (net 11))
   (segment (start 162.56 130.81) (end 163.83 130.81) (width 0.25) (layer F.Cu) (net 11))
+  (segment (start 153.67 151.13) (end 153.67 147.32) (width 0.25) (layer F.Cu) (net 31))
+  (segment (start 163.83 128.27) (end 157.48 128.27) (width 0.25) (layer B.Cu) (net 31))
+  (segment (start 157.48 128.27) (end 153.67 132.08) (width 0.25) (layer B.Cu) (net 31))
+  (via (at 153.67 140.97) (size 0.8) (drill 0.4) (layers F.Cu B.Cu) (net 31))
+  (segment (start 153.67 132.08) (end 153.67 140.97) (width 0.25) (layer B.Cu) (net 31))
+  (segment (start 152.97 147.32) (end 153.67 147.32) (width 0.25) (layer F.Cu) (net 31))
+  (segment (start 151.13 145.48) (end 152.97 147.32) (width 0.25) (layer F.Cu) (net 31))
+  (segment (start 151.13 143.51) (end 151.13 145.48) (width 0.25) (layer F.Cu) (net 31))
+  (segment (start 153.67 140.97) (end 151.13 143.51) (width 0.25) (layer F.Cu) (net 31))
   (zone (net 3) (net_name +12V) (layer B.Cu) (hatch edge 0.508)
     (connect_pads (clearance 0.508))
     (min_thickness 0.254)
-    (fill (arc_segments 32) (thermal_gap 0.508) (thermal_bridge_width 0.508))
+    (fill yes (arc_segments 32) (thermal_gap 0.508) (thermal_bridge_width 0.508))
     (polygon
       (pts
@@
     (connect_pads (clearance 0.508))
     (min_thickness 0.254)
-    (fill (arc_segments 32) (thermal_gap 0.508) (thermal_bridge_width 0.508))
+    (fill yes (arc_segments 32) (thermal_gap 0.508) (thermal_bridge_width 0.508))
     (polygon
       (pts
@@
     (connect_pads (clearance 0.508))
     (min_thickness 0.254)
-    (fill (arc_segments 32) (thermal_gap 0.508) (thermal_bridge_width 0.508))
+    (fill yes (arc_segments 32) (thermal_gap 0.508) (thermal_bridge_width 0.508))
     (polygon
       (pts
@@
     (connect_pads (clearance 0.508))
     (min_thickness 0.254)
-    (fill (arc_segments 32) (thermal_gap 0.508) (thermal_bridge_width 0.508))
+    (fill yes (arc_segments 32) (thermal_gap 0.508) (thermal_bridge_width 0.508))
     (polygon
       (pts
@@
     (connect_pads (clearance 0.508))
     (min_thickness 0.254)
-    (fill (arc_segments 32) (thermal_gap 0.508) (thermal_bridge_width 0.508))
+    (fill yes (arc_segments 32) (thermal_gap 0.508) (thermal_bridge_width 0.508))
     (polygon
       (pts
